Commit message: finished gazebo simulation. Reorganised navigation and launch setup.

File: kmriiwa_description/urdf/kmp200/kmp200.gazebo.xacro (robot description, xacro)
@@ -30,7 +30,7 @@
             <odometryFrame>odom</odometryFrame>
             <odometryRate>20.0</odometryRate>
-            <yaw_velocity_p_gain>1000</yaw_velocity_p_gain>
-            <x_velocity_p_gain>20000</x_velocity_p_gain>
-            <y_velocity_p_gain>20000</y_velocity_p_gain>
+            <yaw_velocity_p_gain>500</yaw_velocity_p_gain>
+            <x_velocity_p_gain>1000</x_velocity_p_gain>
+            <y_velocity_p_gain>1000</y_velocity_p_gain>
         </plugin>
     </gazebo>
@@ -103,4 +103,6 @@
     </gazebo>
     <gazebo reference="front_left_wheel_link">
+        <mu1 value="0.0"/>
+        <mu2 value="0.0"/>
         <surface>
             <contact>
@@ -110,4 +112,6 @@
     </gazebo>
     <gazebo reference="front_right_wheel_link">
+        <mu1 value="0.0"/>
+        <mu2 value="0.0"/>
         <surface>
             <contact>
@@ -117,4 +121,6 @@
     </gazebo>
     <gazebo reference="back_left_wheel_link">
+        <mu1 value="0.0"/>
+        <mu2 value="0.0"/>
         <surface>
             <contact>
@@ -124,4 +130,6 @@
     </gazebo>
     <gazebo reference="back_right_wheel_link">
+        <mu1 value="0.0"/>
+        <mu2 value="0.0"/>
         <surface>
             <contact>

File: kmriiwa_description/urdf/kmp200/kmp200.xacro (robot description, xacro)
@@ -8,5 +8,5 @@
   <xacro:property name="base_width" value="0.63" />
   <xacro:property name="base_mass" value="390" />
-  <xacro:property name="center_of_gravity_height_noload" value="0.16" /> <!-- actual center at 0.26. Changed it to prevent robot rolling over in gazebo with ros_force_based_move plugin-->
+  <xacro:property name="center_of_gravity_height_noload" value="0.26" />
   <xacro:property name="wheel_radius" value="0.125" />
   <xacro:property name="wheel_thickness" value="0.132" />
@@ -37,6 +37,6 @@
             <origin xyz="0 0 ${center_of_gravity_height_noload-ground_clearance}" rpy="0 0 0"/>
             <mass value="${base_mass}"/>
-            <!-- obtained from KMP200 model on fusion 360 with some modification-->
-            <inertia ixx="28.95" ixy="-0.187" ixz="1.242" iyy="44.03" iyz="-0.1441" izz="33.83"/>
+            <!-- obtained from KMP200 model on fusion 360 with some modification to align center of mass with the given one-->
+            <inertia ixx="28.95" ixy="0.0" ixz="0.0" iyy="44.03" iyz="0.0" izz="33.83"/>
         </inertial>
     </link>
