Commit message: added riser flange and reorganised urdf

File: kmriiwa_description/urdf/kmp200/kmp200.xacro (robot description, xacro)
@@ -27,5 +27,5 @@
             <mesh filename="package://kmriiwa_description/meshes/kmp200/KMP200.dae"/>
           </geometry>
-          <material name="Grey"/>
+          <material name="White"/>
         </visual>
         <collision>

Commit message: added nav multi-robot and namespace support

File: kmriiwa_description/urdf/kmp200/kmp200.xacro (robot description, xacro)
@@ -15,11 +15,11 @@
   <xacro:property name="ground_clearance" value="0.025" /> <!-- distance from wheel-floor contact point to base bottom side-->
   <xacro:macro name="kmp200" params="robot_name">
-    <link name="base_footprint"/>
-    <joint name="footprint_to_base_link" type="fixed">
-        <parent link="base_footprint"/>
-        <child link="base_link"/>
+    <link name="${robot_name}_base_footprint"/>
+    <joint name="${robot_name}_footprint_to_base_link" type="fixed">
+        <parent link="${robot_name}_base_footprint"/>
+        <child link="${robot_name}_base_link"/>
         <origin rpy="0 0 0.0" xyz="0 0 ${ground_clearance}"/>
     </joint>
-    <link name="base_link">
+    <link name="${robot_name}_base_link">
     	<origin rpy="0 0 0" xyz="0 0 0"/>
         <visual>
@@ -41,16 +41,16 @@
         </inertial>
     </link>
-    <joint name="base_link_to_top" type="fixed">
-        <parent link="base_link"/>
-        <child link="base_top_link"/>
+    <joint name="${robot_name}_base_link_to_top" type="fixed">
+        <parent link="${robot_name}_base_link"/>
+        <child link="${robot_name}_base_top_link"/>
         <origin rpy="0 0 0.0" xyz="0 0 ${base_height-ground_clearance}"/>
     </joint>
-    <link name="base_top_link"/>
-    <joint name="laser_B1_joint" type="fixed">
-            <parent link="base_link" />
-            <child link="laser_B1_link" />
+    <link name="${robot_name}_base_top_link"/>
+    <joint name="${robot_name}_laser_B1_joint" type="fixed">
+            <parent link="${robot_name}_base_link" />
+            <child link="${robot_name}_laser_B1_link" />
             <origin xyz="0.464 -0.256 0.1168" rpy="0 0 -0.7854"/>
     </joint>
-    <link name="laser_B1_link">
+    <link name="${robot_name}_laser_B1_link">
         <visual>
           <origin xyz="0 0 0" rpy="3.1413 0 0"/>
@@ -71,10 +71,10 @@
         </inertial>
     </link>
-    <joint name="laser_B4_joint" type="fixed">
-            <parent link="base_link" />
-            <child link="laser_B4_link" />
+    <joint name="${robot_name}_laser_B4_joint" type="fixed">
+            <parent link="${robot_name}_base_link" />
+            <child link="${robot_name}_laser_B4_link" />
             <origin xyz="-0.464 0.256 0.1168" rpy="0 0 2.3562"/>
     </joint>
-    <link name="laser_B4_link">
+    <link name="${robot_name}_laser_B4_link">
         <visual>
           <origin xyz="0.0 0 0" rpy="0 3.1413 3.1413"/>
@@ -95,5 +95,5 @@
         </inertial>
     </link>
-    <link name="front_left_wheel_link">
+    <link name="${robot_name}_front_left_wheel_link">
         <visual>
           <origin xyz="0 0 0" rpy="0 0 0" />
@@ -109,5 +109,5 @@
         </collision>
     </link>
-    <link name="front_right_wheel_link">
+    <link name="${robot_name}_front_right_wheel_link">
         <visual>
           <origin xyz="0 0 0" rpy="0 0 0" />
@@ -123,5 +123,5 @@
         </collision>
     </link>
-    <link name="back_left_wheel_link">
+    <link name="${robot_name}_back_left_wheel_link">
         <visual>
           <origin xyz="0 0 0" rpy="0 0 0" />
@@ -137,5 +137,5 @@
         </collision>
     </link>
-    <link name="back_right_wheel_link">
+    <link name="${robot_name}_back_right_wheel_link">
         <visual>
           <origin xyz="0 0 0" rpy="0 0 0" />
@@ -155,7 +155,7 @@
         </inertial> -->
     </link>
-    <joint name="front_left_wheel_joint" type="fixed">
-        <parent link="base_link"/>
-        <child link="front_left_wheel_link"/>
+    <joint name="${robot_name}_front_left_wheel_joint" type="fixed">
+        <parent link="${robot_name}_base_link"/>
+        <child link="${robot_name}_front_left_wheel_link"/>
         <axis xyz="0 1 0"/>
         <origin xyz="${wheel_base/2} ${track_gauge/2} ${wheel_radius-ground_clearance}"/>
@@ -163,7 +163,7 @@
         <joint_properties damping="0.0" friction="0.0"/>
     </joint>
-    <joint name="front_right_wheel_joint" type="fixed">
-        <parent link="base_link"/>
-        <child link="front_right_wheel_link"/>
+    <joint name="${robot_name}_front_right_wheel_joint" type="fixed">
+        <parent link="${robot_name}_base_link"/>
+        <child link="${robot_name}_front_right_wheel_link"/>
         <origin xyz="${wheel_base/2} ${-1*track_gauge/2} ${wheel_radius-ground_clearance}"/>
         <axis xyz="0 1 0"/>
@@ -171,7 +171,7 @@
         <joint_properties damping="0.0" friction="0.0"/>
     </joint>
-    <joint name="back_left_wheel_joint" type="fixed">
-        <parent link="base_link"/>
-        <child link="back_left_wheel_link"/>
+    <joint name="${robot_name}_back_left_wheel_joint" type="fixed">
+        <parent link="${robot_name}_base_link"/>
+        <child link="${robot_name}_back_left_wheel_link"/>
         <origin xyz="${-1*wheel_base/2} ${track_gauge/2} ${wheel_radius-ground_clearance}"/>
         <axis xyz="0 1 0"/>
@@ -179,7 +179,7 @@
         <joint_properties damping="0.0" friction="0.0"/>
     </joint>
-    <joint name="back_right_wheel_joint" type="fixed">
-        <parent link="base_link"/>
-        <child link="back_right_wheel_link"/>
+    <joint name="${robot_name}_back_right_wheel_joint" type="fixed">
+        <parent link="${robot_name}_base_link"/>
+        <child link="${robot_name}_back_right_wheel_link"/>
         <origin xyz="${-1*wheel_base/2} ${-1*track_gauge/2} ${wheel_radius-ground_clearance}"/>
         <axis xyz="0 1 0"/>

File: kmriiwa_description/urdf/robot/kmriiwa.urdf.xacro (robot description, xacro)
@@ -21,10 +21,10 @@
   <xacro:kmp200 robot_name="$(arg robot_name)"/>
    <!--riser flange-->
-  <joint name="base_top_riser_flange_joint" type="fixed">
-        <parent link="base_top_link"/>
-        <child link="riser_flange_link"/>
+  <joint name="$(arg robot_name)_base_top_riser_flange_joint" type="fixed">
+        <parent link="$(arg robot_name)_base_top_link"/>
+        <child link="$(arg robot_name)_riser_flange_link"/>
         <origin xyz="${flange_origin_xyz}" rpy="${flange_origin_rpy}"/>
   </joint>
-  <link name="riser_flange_link">
+  <link name="$(arg robot_name)_riser_flange_link">
       <visual>
         <origin xyz="0 0 0" rpy="0 0 0" />
@@ -42,5 +42,5 @@
   </link>
   <!--iiwa-->
-  <xacro:iiwa14 hardware_interface="$(arg hardware_interface)" robot_name="$(arg robot_name)" parent="riser_flange_link">
+  <xacro:iiwa14 hardware_interface="$(arg hardware_interface)" robot_name="$(arg robot_name)" parent="$(arg robot_name)_riser_flange_link">
     <origin xyz="0 0 ${riser_flange_height/2}" rpy="0 0 0" />
   </xacro:iiwa14>
