Commit message: can simulate robot in gazebo. Fixed description bugs.

File: kmriiwa_description/urdf/iiwa14/iiwa14.xacro (robot description, xacro)
@@ -2,9 +2,9 @@
 <robot xmlns:xacro="http://www.ros.org/wiki/xacro">
   <!-- Import all Gazebo-customization elements, including Gazebo colors -->
-  <xacro:include filename="$(find iiwa_description)/urdf/iiwa.gazebo.xacro" />
+  <xacro:include filename="$(find kmriiwa_description)/urdf/iiwa14/iiwa.gazebo.xacro" />
   <!-- Import Transmissions -->
-  <xacro:include filename="$(find iiwa_description)/urdf/iiwa.transmission.xacro" />
+  <xacro:include filename="$(find kmriiwa_description)/urdf/iiwa14/iiwa.transmission.xacro" />
   <!-- Include Utilities -->
-  <xacro:include filename="$(find iiwa_description)/urdf/utilities.xacro" />
+  <xacro:include filename="$(find kmriiwa_description)/urdf/iiwa14/utilities.xacro" />
   <!-- some constants -->
   <xacro:property name="safety_controller_k_pos" value="100" />
@@ -22,5 +22,5 @@
     <link name="${robot_name}_link_0">
       <inertial>
-        <origin xyz="-0.1 0 0.07" rpy="0 0 0"/>
+        <origin xyz="0.0 0.0 0.0" rpy="0 0 0"/>
         <mass value="5"/>
         <inertia ixx="0.05"  ixy="0"  ixz="0" iyy="0.06" iyz="0" izz="0.03" />
@@ -29,5 +29,5 @@
         <origin xyz="0 0 0" rpy="0 0 0"/>
         <geometry>
-          <mesh filename="package://iiwa_description/meshes/iiwa14/visual/link_0.stl"/>
+          <mesh filename="package://kmriiwa_description/meshes/iiwa14/visual/link_0.stl"/>
         </geometry>
         <material name="Grey"/>
@@ -36,5 +36,5 @@
         <origin xyz="0 0 0" rpy="0 0 0"/>
         <geometry>
-          <mesh filename="package://iiwa_description/meshes/iiwa14/collision/link_0.stl"/>
+          <mesh filename="package://kmriiwa_description/meshes/iiwa14/collision/link_0.stl"/>
         </geometry>
         <material name="Grey"/>
@@ -70,12 +70,12 @@
         <origin xyz="0 0 0" rpy="0 0 0"/>
         <geometry>
-          <mesh filename="package://iiwa_description/meshes/iiwa14/visual/link_1.stl"/>
-        </geometry>
-        <material name="Orange"/>
-      </visual>
-      <collision>
-        <origin xyz="0 0 0" rpy="0 0 0"/>
-        <geometry>
-          <mesh filename="package://iiwa_description/meshes/iiwa14/collision/link_1.stl"/>
+          <mesh filename="package://kmriiwa_description/meshes/iiwa14/visual/link_1.stl"/>
+        </geometry>
+        <material name="Orange"/>
+      </visual>
+      <collision>
+        <origin xyz="0 0 0" rpy="0 0 0"/>
+        <geometry>
+          <mesh filename="package://kmriiwa_description/meshes/iiwa14/collision/link_1.stl"/>
         </geometry>
         <material name="Orange"/>
@@ -105,12 +105,12 @@
         <origin xyz="0 0 0" rpy="0 0 0"/>
         <geometry>
-          <mesh filename="package://iiwa_description/meshes/iiwa14/visual/link_2.stl"/>
-        </geometry>
-        <material name="Orange"/>
-      </visual>
-      <collision>
-        <origin xyz="0 0 0" rpy="0 0 0"/>
-        <geometry>
-          <mesh filename="package://iiwa_description/meshes/iiwa14/collision/link_2.stl"/>
+          <mesh filename="package://kmriiwa_description/meshes/iiwa14/visual/link_2.stl"/>
+        </geometry>
+        <material name="Orange"/>
+      </visual>
+      <collision>
+        <origin xyz="0 0 0" rpy="0 0 0"/>
+        <geometry>
+          <mesh filename="package://kmriiwa_description/meshes/iiwa14/collision/link_2.stl"/>
         </geometry>
         <material name="Orange"/>
@@ -140,12 +140,12 @@
         <origin xyz="0 0 0" rpy="0 0 0"/>
         <geometry>
-          <mesh filename="package://iiwa_description/meshes/iiwa14/visual/link_3.stl"/>
-        </geometry>
-        <material name="Orange"/>
-      </visual>
-      <collision>
-        <origin xyz="0 0 0" rpy="0 0 0"/>
-        <geometry>
-          <mesh filename="package://iiwa_description/meshes/iiwa14/collision/link_3.stl"/>
+          <mesh filename="package://kmriiwa_description/meshes/iiwa14/visual/link_3.stl"/>
+        </geometry>
+        <material name="Orange"/>
+      </visual>
+      <collision>
+        <origin xyz="0 0 0" rpy="0 0 0"/>
+        <geometry>
+          <mesh filename="package://kmriiwa_description/meshes/iiwa14/collision/link_3.stl"/>
         </geometry>
         <material name="Orange"/>
@@ -175,12 +175,12 @@
         <origin xyz="0 0 0" rpy="0 0 0"/>
         <geometry>
-          <mesh filename="package://iiwa_description/meshes/iiwa14/visual/link_4.stl"/>
-        </geometry>
-        <material name="Orange"/>
-      </visual>
-      <collision>
-        <origin xyz="0 0 0" rpy="0 0 0"/>
-        <geometry>
-          <mesh filename="package://iiwa_description/meshes/iiwa14/collision/link_4.stl"/>
+          <mesh filename="package://kmriiwa_description/meshes/iiwa14/visual/link_4.stl"/>
+        </geometry>
+        <material name="Orange"/>
+      </visual>
+      <collision>
+        <origin xyz="0 0 0" rpy="0 0 0"/>
+        <geometry>
+          <mesh filename="package://kmriiwa_description/meshes/iiwa14/collision/link_4.stl"/>
         </geometry>
         <material name="Orange"/>
@@ -210,12 +210,12 @@
         <origin xyz="0 0 0" rpy="0 0 0"/>
         <geometry>
-          <mesh filename="package://iiwa_description/meshes/iiwa14/visual/link_5.stl"/>
-        </geometry>
-        <material name="Orange"/>
-      </visual>
-      <collision>
-        <origin xyz="0 0 0" rpy="0 0 0"/>
-        <geometry>
-          <mesh filename="package://iiwa_description/meshes/iiwa14/collision/link_5.stl"/>
+          <mesh filename="package://kmriiwa_description/meshes/iiwa14/visual/link_5.stl"/>
+        </geometry>
+        <material name="Orange"/>
+      </visual>
+      <collision>
+        <origin xyz="0 0 0" rpy="0 0 0"/>
+        <geometry>
+          <mesh filename="package://kmriiwa_description/meshes/iiwa14/collision/link_5.stl"/>
         </geometry>
         <material name="Orange"/>
@@ -245,12 +245,12 @@
         <origin xyz="0 0 0" rpy="0 0 0"/>
         <geometry>
-          <mesh filename="package://iiwa_description/meshes/iiwa14/visual/link_6.stl"/>
-        </geometry>
-        <material name="Orange"/>
-      </visual>
-      <collision>
-        <origin xyz="0 0 0" rpy="0 0 0"/>
-        <geometry>
-          <mesh filename="package://iiwa_description/meshes/iiwa14/collision/link_6.stl"/>
+          <mesh filename="package://kmriiwa_description/meshes/iiwa14/visual/link_6.stl"/>
+        </geometry>
+        <material name="Orange"/>
+      </visual>
+      <collision>
+        <origin xyz="0 0 0" rpy="0 0 0"/>
+        <geometry>
+          <mesh filename="package://kmriiwa_description/meshes/iiwa14/collision/link_6.stl"/>
         </geometry>
         <material name="Orange"/>
@@ -280,5 +280,5 @@
         <origin xyz="0 0 0" rpy="0 0 0"/>
         <geometry>
-          <mesh filename="package://iiwa_description/meshes/iiwa14/visual/link_7.stl"/>
+          <mesh filename="package://kmriiwa_description/meshes/iiwa14/visual/link_7.stl"/>
         </geometry>
         <material name="Grey"/>
@@ -287,5 +287,5 @@
         <origin xyz="0 0 0" rpy="0 0 0"/>
         <geometry>
-          <mesh filename="package://iiwa_description/meshes/iiwa14/collision/link_7.stl"/>
+          <mesh filename="package://kmriiwa_description/meshes/iiwa14/collision/link_7.stl"/>
         </geometry>
         <material name="Grey"/>

File: kmriiwa_description/urdf/kmp200/kmp200.xacro (robot description, xacro)
@@ -1,10 +1,23 @@
 <?xml version="1.0"?>
 <robot xmlns:xacro="http://www.ros.org/wiki/xacro">
-  <xacro:macro name="kmp200">
+  <!-- Import Gazebo-settings -->
+  <xacro:include filename="$(find kmriiwa_description)/urdf/kmp200/kmp200.gazebo.xacro" />
+  <!-- some technical data constants obtained from KMP200 manual-->
+  <xacro:property name="base_length" value="1.08" />
+  <xacro:property name="base_height" value="0.7" />
+  <xacro:property name="base_width" value="0.63" />
+  <xacro:property name="base_mass" value="390" />
+  <xacro:property name="center_of_gravity_height_noload" value="0.16" /> <!-- actual center at 0.26. Changed it to prevent robot rolling over in gazebo with ros_force_based_move plugin-->
+  <xacro:property name="wheel_radius" value="0.125" />
+  <xacro:property name="wheel_thickness" value="0.132" />
+  <xacro:property name="track_gauge" value="0.365" />
+  <xacro:property name="wheel_base" value="0.56" />
+  <xacro:property name="ground_clearance" value="0.025" /> <!-- distance from wheel-floor contact point to base bottom side-->
+  <xacro:macro name="kmp200" params="robot_name">
     <link name="base_footprint"/>
     <joint name="footprint_to_base_link" type="fixed">
         <parent link="base_footprint"/>
         <child link="base_link"/>
-        <origin rpy="0 0 0.0" xyz="0 0 0.033"/>
+        <origin rpy="0 0 0.0" xyz="0 0 ${ground_clearance}"/>
     </joint>
     <link name="base_link">
@@ -18,12 +31,18 @@
         <collision>
           <geometry>
-            <box size="1.12 0.63 0.7"/>
+            <mesh filename="package://kmriiwa_description/meshes/kmp200/KMP200.dae"/>
           </geometry>
         </collision>
+        <inertial>
+            <origin xyz="0 0 ${center_of_gravity_height_noload-ground_clearance}" rpy="0 0 0"/>
+            <mass value="${base_mass}"/>
+            <!-- obtained from KMP200 model on fusion 360 with some modification-->
+            <inertia ixx="28.95" ixy="-0.187" ixz="1.242" iyy="44.03" iyz="-0.1441" izz="33.83"/>
+        </inertial>
     </link>
     <joint name="base_link_to_top" type="fixed">
         <parent link="base_link"/>
         <child link="base_top_link"/>
-        <origin rpy="0 0 0.0" xyz="0 0 0.6672"/>
+        <origin rpy="0 0 0.0" xyz="0 0 ${base_height-ground_clearance}"/>
     </joint>
     <link name="base_top_link"/>
@@ -78,7 +97,7 @@
     <link name="front_left_wheel_link">
         <visual>
-          <origin xyz="0 0 0" rpy="1.57 0 0" />
+          <origin xyz="0 0 0" rpy="0 0 0" />
           <geometry>
-            <cylinder length="0.132" radius="0.125" />
+            <mesh filename="package://kmriiwa_description/meshes/kmp200/wheels/omni_wheel_1.dae" scale="1.06695 1.06695 1.06695"/>
           </geometry>
         </visual>
@@ -86,5 +105,5 @@
           <origin xyz="0 0 0" rpy="1.57 0 0" />
           <geometry>
-            <cylinder length="0.132" radius="0.125" />
+            <cylinder length="${wheel_thickness}" radius="${wheel_radius}" />
           </geometry>
         </collision>
@@ -92,7 +111,7 @@
     <link name="front_right_wheel_link">
         <visual>
-          <origin xyz="0 0 0" rpy="1.57 0 0" />
+          <origin xyz="0 0 0" rpy="0 0 0" />
           <geometry>
-            <cylinder length="0.132" radius="0.125" />
+            <mesh filename="package://kmriiwa_description/meshes/kmp200/wheels/omni_wheel_1.dae" scale="1.06695 1.06695 1.06695"/>
           </geometry>
         </visual>
@@ -100,5 +119,5 @@
           <origin xyz="0 0 0" rpy="1.57 0 0" />
           <geometry>
-            <cylinder length="0.132" radius="0.125" />
+            <cylinder length="${wheel_thickness}" radius="${wheel_radius}" />
           </geometry>
         </collision>
@@ -106,7 +125,7 @@
     <link name="back_left_wheel_link">
         <visual>
-          <origin xyz="0 0 0" rpy="1.57 0 0" />
+          <origin xyz="0 0 0" rpy="0 0 0" />
           <geometry>
-            <cylinder length="0.132" radius="0.125" />
+            <mesh filename="package://kmriiwa_description/meshes/kmp200/wheels/omni_wheel_1.dae" scale="1.06695 1.06695 1.06695"/>
           </geometry>
         </visual>
@@ -114,5 +133,5 @@
           <origin xyz="0 0 0" rpy="1.57 0 0" />
           <geometry>
-            <cylinder length="0.132" radius="0.125" />
+            <cylinder length="${wheel_thickness}" radius="${wheel_radius}" />
           </geometry>
         </collision>
@@ -120,7 +139,7 @@
     <link name="back_right_wheel_link">
         <visual>
-          <origin xyz="0 0 0" rpy="1.57 0 0" />
+          <origin xyz="0 0 0" rpy="0 0 0" />
           <geometry>
-            <cylinder length="0.132" radius="0.125" />
+            <mesh filename="package://kmriiwa_description/meshes/kmp200/wheels/omni_wheel_1.dae" scale="1.06695 1.06695 1.06695"/>
           </geometry>
         </visual>
@@ -128,7 +147,11 @@
           <origin xyz="0 0 0" rpy="1.57 0 0" />
           <geometry>
-            <cylinder length="0.132" radius="0.125" />
+            <cylinder length="${wheel_thickness}" radius="${wheel_radius}" />
           </geometry>
         </collision>
+        <!-- <inertial>
+            <mass value="14"/>
+            <inertia ixx="0.075016" ixy="0.0" ixz="0.0" iyy="0.075016" iyz="0.0" izz="0.109375"/>
+        </inertial> -->
     </link>
     <joint name="front_left_wheel_joint" type="fixed">
@@ -136,5 +159,5 @@
         <child link="front_left_wheel_link"/>
         <axis xyz="0 1 0"/>
-        <origin xyz="0.28 0.182 0.092"/>
+        <origin xyz="${wheel_base/2} ${track_gauge/2} ${wheel_radius-ground_clearance}"/>
         <limit effort="100" velocity="100"/>
         <joint_properties damping="0.0" friction="0.0"/>
@@ -143,5 +166,5 @@
         <parent link="base_link"/>
         <child link="front_right_wheel_link"/>
-        <origin xyz="0.28 -0.182 0.092"/>
+        <origin xyz="${wheel_base/2} ${-1*track_gauge/2} ${wheel_radius-ground_clearance}"/>
         <axis xyz="0 1 0"/>
         <limit effort="100" velocity="100"/>
@@ -151,5 +174,5 @@
         <parent link="base_link"/>
         <child link="back_left_wheel_link"/>
-        <origin xyz="-0.28 0.182 0.092"/>
+        <origin xyz="${-1*wheel_base/2} ${track_gauge/2} ${wheel_radius-ground_clearance}"/>
         <axis xyz="0 1 0"/>
         <limit effort="100" velocity="100"/>
@@ -159,9 +182,11 @@
         <parent link="base_link"/>
         <child link="back_right_wheel_link"/>
-        <origin xyz="-0.28 -0.182 0.092"/>
+        <origin xyz="${-1*wheel_base/2} ${-1*track_gauge/2} ${wheel_radius-ground_clearance}"/>
         <axis xyz="0 1 0"/>
         <limit effort="100" velocity="100"/>
         <joint_properties damping="0.0" friction="0.0"/>
     </joint>
+    <!--Extensions -->
+    <xacro:kmp200_gazebo robot_name="${robot_name}"/>
    </xacro:macro>
 </robot>

File: kmriiwa_description/urdf/kmriiwa.urdf.xacro (robot description, xacro)
@@ -7,13 +7,18 @@
   <!--Import the kmp200 macro -->
   <xacro:include filename="$(find kmriiwa_description)/urdf/kmp200/kmp200.xacro"/>
+  <xacro:property name="arm_base_flange_x_pos" value="0.363" />
+  <xacro:property name="arm_base_flange_y_pos" value="-0.184" />
+  <xacro:property name="arm_base_flange_z_pos" value="-0.01" />
+  <xacro:property name="arm_base_flange_yew" value="-1.5708" />
+  <xacro:property name="origin_xyz" value="${arm_base_flange_x_pos} ${arm_base_flange_y_pos} ${arm_base_flange_z_pos}"/>
+  <xacro:property name="origin_rpy" value="0 0 ${arm_base_flange_yew}"/>
+  <xacro:arg name="robot_name" default="kmriiwa"/>
+  <xacro:arg name="hardware_interface" default="PositionJointInterface"/>
   <!--kmp200-->
-  <xacro:kmp200/>
+  <xacro:kmp200 robot_name="$(arg robot_name)"/>
+  <!--TODO add joint and link for the extra flange-->
   <!--iiwa-->
-  <xacro:arg name="hardware_interface" default="PositionJointInterface"/>
-  <xacro:arg name="robot_name" default="kmriiwa_iiwa"/>
-  <xacro:arg name="origin_xyz" default="0.363 -0.184 0.0"/>
-  <xacro:arg name="origin_rpy" default="0 0 -1.5708"/>
   <xacro:iiwa14 hardware_interface="$(arg hardware_interface)" robot_name="$(arg robot_name)" parent="base_top_link">
-    <origin xyz="$(arg origin_xyz)" rpy="$(arg origin_rpy)" />
+    <origin xyz="${origin_xyz}" rpy="${origin_rpy}" />
   </xacro:iiwa14>
 </robot>

Commit message: moveit_ns_added

File: kmriiwa_description/urdf/iiwa14/iiwa14.xacro (robot description, xacro)
@@ -15,10 +15,10 @@
   <xacro:macro name="iiwa14" params="parent hardware_interface robot_name *origin">
     <!--joint between {parent} and link_0-->
-    <joint name="${parent}_${robot_name}_joint" type="fixed">
+    <joint name="${parent}_kmriiwa_joint" type="fixed">
       <xacro:insert_block name="origin"/>
       <parent link="${parent}"/>
-      <child link="${robot_name}_link_0"/>
-    </joint>
-    <link name="${robot_name}_link_0">
+      <child link="kmriiwa_link_0"/>
+    </joint>
+    <link name="kmriiwa_link_0">
       <inertial>
         <origin xyz="0.0 0.0 0.0" rpy="0 0 0"/>
@@ -48,7 +48,7 @@
     </link>
     <!-- joint between link_0 and link_1 -->
-    <joint name="${robot_name}_joint_1" type="revolute">
-      <parent link="${robot_name}_link_0"/>
-      <child link="${robot_name}_link_1"/>
+    <joint name="kmriiwa_joint_1" type="revolute">
+      <parent link="kmriiwa_link_0"/>
+      <child link="kmriiwa_link_1"/>
       <origin xyz="0 0 0.1575" rpy="0 0 0"/>
       <axis xyz="0 0 1"/>
@@ -61,5 +61,5 @@
       <dynamics damping="${joint_damping}"/>
     </joint>
-    <link name="${robot_name}_link_1">
+    <link name="kmriiwa_link_1">
       <inertial>
         <origin xyz="0 -0.03 0.12" rpy="0 0 0"/>
@@ -83,7 +83,7 @@
     </link>
     <!-- joint between link_1 and link_2 -->
-    <joint name="${robot_name}_joint_2" type="revolute">
-      <parent link="${robot_name}_link_1"/>
-      <child link="${robot_name}_link_2"/>
+    <joint name="kmriiwa_joint_2" type="revolute">
+      <parent link="kmriiwa_link_1"/>
+      <child link="kmriiwa_link_2"/>
       <origin xyz="0 0 0.2025" rpy="${PI / 2}   0 ${PI}"/>
       <axis xyz="0 0 1"/>
@@ -96,5 +96,5 @@
       <dynamics damping="${joint_damping}"/>
     </joint>
-    <link name="${robot_name}_link_2">
+    <link name="kmriiwa_link_2">
       <inertial>
         <origin xyz="0.0003 0.059 0.042" rpy="0 0 0"/>
@@ -118,7 +118,7 @@
     </link>
     <!-- joint between link_2 and link_3 -->
-    <joint name="${robot_name}_joint_3" type="revolute">
-      <parent link="${robot_name}_link_2"/>
-      <child link="${robot_name}_link_3"/>
+    <joint name="kmriiwa_joint_3" type="revolute">
+      <parent link="kmriiwa_link_2"/>
+      <child link="kmriiwa_link_3"/>
       <origin xyz="0 0.2045 0" rpy="${PI / 2} 0 ${PI}"/>
       <axis xyz="0 0 1"/>
@@ -131,5 +131,5 @@
       <dynamics damping="${joint_damping}"/>
     </joint>
-    <link name="${robot_name}_link_3">
+    <link name="kmriiwa_link_3">
       <inertial>
         <origin xyz="0 0.03 0.13" rpy="0 0 0"/>
@@ -153,7 +153,7 @@
     </link>
     <!-- joint between link_3 and link_4 -->
-    <joint name="${robot_name}_joint_4" type="revolute">
-      <parent link="${robot_name}_link_3"/>
-      <child link="${robot_name}_link_4"/>
+    <joint name="kmriiwa_joint_4" type="revolute">
+      <parent link="kmriiwa_link_3"/>
+      <child link="kmriiwa_link_4"/>
       <origin xyz="0 0 0.2155" rpy="${PI / 2} 0 0"/>
       <axis xyz="0 0 1"/>
@@ -166,5 +166,5 @@
       <dynamics damping="${joint_damping}"/>
     </joint>
-    <link name="${robot_name}_link_4">
+    <link name="kmriiwa_link_4">
       <inertial>
         <origin xyz="0 0.067 0.034" rpy="0 0 0"/>
@@ -188,7 +188,7 @@
     </link>
     <!-- joint between link_4 and link_5 -->
-    <joint name="${robot_name}_joint_5" type="revolute">
-      <parent link="${robot_name}_link_4"/>
-      <child link="${robot_name}_link_5"/>
+    <joint name="kmriiwa_joint_5" type="revolute">
+      <parent link="kmriiwa_link_4"/>
+      <child link="kmriiwa_link_5"/>
       <origin xyz="0 0.1845 0" rpy="${-PI / 2} ${PI} 0"/>
       <axis xyz="0 0 1"/>
@@ -201,5 +201,5 @@
       <dynamics damping="${joint_damping}"/>
     </joint>
-    <link name="${robot_name}_link_5">
+    <link name="kmriiwa_link_5">
       <inertial>
         <origin xyz="0.0001 0.021 0.076" rpy="0 0 0"/>
@@ -223,7 +223,7 @@
     </link>
     <!-- joint between link_5 and link_6 -->
-    <joint name="${robot_name}_joint_6" type="revolute">
-      <parent link="${robot_name}_link_5"/>
-      <child link="${robot_name}_link_6"/>
+    <joint name="kmriiwa_joint_6" type="revolute">
+      <parent link="kmriiwa_link_5"/>
+      <child link="kmriiwa_link_6"/>
       <origin xyz="0 0 0.2155" rpy="${PI / 2} 0 0"/>
       <axis xyz="0 0 1"/>
@@ -236,5 +236,5 @@
       <dynamics damping="${joint_damping}"/>
     </joint>
-    <link name="${robot_name}_link_6">
+    <link name="kmriiwa_link_6">
       <inertial>
         <origin xyz="0 0.0006 0.0004" rpy="0 0 0"/>
@@ -258,7 +258,7 @@
     </link>
     <!-- joint between link_6 and link_7 -->
-    <joint name="${robot_name}_joint_7" type="revolute">
-      <parent link="${robot_name}_link_6"/>
-      <child link="${robot_name}_link_7"/>
+    <joint name="kmriiwa_joint_7" type="revolute">
+      <parent link="kmriiwa_link_6"/>
+      <child link="kmriiwa_link_7"/>
       <origin xyz="0 0.081 0" rpy="${- PI / 2} ${PI} 0"/>
       <axis xyz="0 0 1"/>
@@ -271,5 +271,5 @@
       <dynamics damping="${joint_damping}"/>
     </joint>
-    <link name="${robot_name}_link_7">
+    <link name="kmriiwa_link_7">
       <inertial>
         <origin xyz="0 0 0.02" rpy="0 0 0"/>
@@ -292,10 +292,10 @@
       </collision>
     </link>
-    <joint name="${robot_name}_joint_ee" type="fixed">
-      <parent link="${robot_name}_link_7"/>
-      <child link="${robot_name}_link_ee"/>
+    <joint name="kmriiwa_joint_ee" type="fixed">
+      <parent link="kmriiwa_link_7"/>
+      <child link="kmriiwa_link_ee"/>
       <origin xyz="0 0 0.045" rpy="0 0 0"/>
     </joint>
-    <link name="${robot_name}_link_ee">
+    <link name="kmriiwa_link_ee">
     </link>
     <!--Extensions -->
