Commit message: added moveit namespace and multi-robot support

File: kmriiwa_description/urdf/iiwa14/iiwa14.xacro (robot description, xacro)
@@ -15,10 +15,10 @@
   <xacro:macro name="iiwa14" params="parent hardware_interface robot_name *origin">
     <!--joint between {parent} and link_0-->
-    <joint name="${parent}_kmriiwa_joint" type="fixed">
+    <joint name="${parent}_${robot_name}_joint" type="fixed">
       <xacro:insert_block name="origin"/>
       <parent link="${parent}"/>
-      <child link="kmriiwa_link_0"/>
-    </joint>
-    <link name="kmriiwa_link_0">
+      <child link="${robot_name}_link_0"/>
+    </joint>
+    <link name="${robot_name}_link_0">
       <inertial>
         <origin xyz="0.0 0.0 0.0" rpy="0 0 0"/>
@@ -48,7 +48,7 @@
     </link>
     <!-- joint between link_0 and link_1 -->
-    <joint name="kmriiwa_joint_1" type="revolute">
-      <parent link="kmriiwa_link_0"/>
-      <child link="kmriiwa_link_1"/>
+    <joint name="${robot_name}_joint_1" type="revolute">
+      <parent link="${robot_name}_link_0"/>
+      <child link="${robot_name}_link_1"/>
       <origin xyz="0 0 0.1575" rpy="0 0 0"/>
       <axis xyz="0 0 1"/>
@@ -61,5 +61,5 @@
       <dynamics damping="${joint_damping}"/>
     </joint>
-    <link name="kmriiwa_link_1">
+    <link name="${robot_name}_link_1">
       <inertial>
         <origin xyz="0 -0.03 0.12" rpy="0 0 0"/>
@@ -83,7 +83,7 @@
     </link>
     <!-- joint between link_1 and link_2 -->
-    <joint name="kmriiwa_joint_2" type="revolute">
-      <parent link="kmriiwa_link_1"/>
-      <child link="kmriiwa_link_2"/>
+    <joint name="${robot_name}_joint_2" type="revolute">
+      <parent link="${robot_name}_link_1"/>
+      <child link="${robot_name}_link_2"/>
       <origin xyz="0 0 0.2025" rpy="${PI / 2}   0 ${PI}"/>
       <axis xyz="0 0 1"/>
@@ -96,5 +96,5 @@
       <dynamics damping="${joint_damping}"/>
     </joint>
-    <link name="kmriiwa_link_2">
+    <link name="${robot_name}_link_2">
       <inertial>
         <origin xyz="0.0003 0.059 0.042" rpy="0 0 0"/>
@@ -118,7 +118,7 @@
     </link>
     <!-- joint between link_2 and link_3 -->
-    <joint name="kmriiwa_joint_3" type="revolute">
-      <parent link="kmriiwa_link_2"/>
-      <child link="kmriiwa_link_3"/>
+    <joint name="${robot_name}_joint_3" type="revolute">
+      <parent link="${robot_name}_link_2"/>
+      <child link="${robot_name}_link_3"/>
       <origin xyz="0 0.2045 0" rpy="${PI / 2} 0 ${PI}"/>
       <axis xyz="0 0 1"/>
@@ -131,5 +131,5 @@
       <dynamics damping="${joint_damping}"/>
     </joint>
-    <link name="kmriiwa_link_3">
+    <link name="${robot_name}_link_3">
       <inertial>
         <origin xyz="0 0.03 0.13" rpy="0 0 0"/>
@@ -153,7 +153,7 @@
     </link>
     <!-- joint between link_3 and link_4 -->
-    <joint name="kmriiwa_joint_4" type="revolute">
-      <parent link="kmriiwa_link_3"/>
-      <child link="kmriiwa_link_4"/>
+    <joint name="${robot_name}_joint_4" type="revolute">
+      <parent link="${robot_name}_link_3"/>
+      <child link="${robot_name}_link_4"/>
       <origin xyz="0 0 0.2155" rpy="${PI / 2} 0 0"/>
       <axis xyz="0 0 1"/>
@@ -166,5 +166,5 @@
       <dynamics damping="${joint_damping}"/>
     </joint>
-    <link name="kmriiwa_link_4">
+    <link name="${robot_name}_link_4">
       <inertial>
         <origin xyz="0 0.067 0.034" rpy="0 0 0"/>
@@ -188,7 +188,7 @@
     </link>
     <!-- joint between link_4 and link_5 -->
-    <joint name="kmriiwa_joint_5" type="revolute">
-      <parent link="kmriiwa_link_4"/>
-      <child link="kmriiwa_link_5"/>
+    <joint name="${robot_name}_joint_5" type="revolute">
+      <parent link="${robot_name}_link_4"/>
+      <child link="${robot_name}_link_5"/>
       <origin xyz="0 0.1845 0" rpy="${-PI / 2} ${PI} 0"/>
       <axis xyz="0 0 1"/>
@@ -201,5 +201,5 @@
       <dynamics damping="${joint_damping}"/>
     </joint>
-    <link name="kmriiwa_link_5">
+    <link name="${robot_name}_link_5">
       <inertial>
         <origin xyz="0.0001 0.021 0.076" rpy="0 0 0"/>
@@ -223,7 +223,7 @@
     </link>
     <!-- joint between link_5 and link_6 -->
-    <joint name="kmriiwa_joint_6" type="revolute">
-      <parent link="kmriiwa_link_5"/>
-      <child link="kmriiwa_link_6"/>
+    <joint name="${robot_name}_joint_6" type="revolute">
+      <parent link="${robot_name}_link_5"/>
+      <child link="${robot_name}_link_6"/>
       <origin xyz="0 0 0.2155" rpy="${PI / 2} 0 0"/>
       <axis xyz="0 0 1"/>
@@ -236,5 +236,5 @@
       <dynamics damping="${joint_damping}"/>
     </joint>
-    <link name="kmriiwa_link_6">
+    <link name="${robot_name}_link_6">
       <inertial>
         <origin xyz="0 0.0006 0.0004" rpy="0 0 0"/>
@@ -258,7 +258,7 @@
     </link>
     <!-- joint between link_6 and link_7 -->
-    <joint name="kmriiwa_joint_7" type="revolute">
-      <parent link="kmriiwa_link_6"/>
-      <child link="kmriiwa_link_7"/>
+    <joint name="${robot_name}_joint_7" type="revolute">
+      <parent link="${robot_name}_link_6"/>
+      <child link="${robot_name}_link_7"/>
       <origin xyz="0 0.081 0" rpy="${- PI / 2} ${PI} 0"/>
       <axis xyz="0 0 1"/>
@@ -271,5 +271,5 @@
       <dynamics damping="${joint_damping}"/>
     </joint>
-    <link name="kmriiwa_link_7">
+    <link name="${robot_name}_link_7">
       <inertial>
         <origin xyz="0 0 0.02" rpy="0 0 0"/>
@@ -292,10 +292,10 @@
       </collision>
     </link>
-    <joint name="kmriiwa_joint_ee" type="fixed">
-      <parent link="kmriiwa_link_7"/>
-      <child link="kmriiwa_link_ee"/>
+    <joint name="${robot_name}_joint_ee" type="fixed">
+      <parent link="${robot_name}_link_7"/>
+      <child link="${robot_name}_link_ee"/>
       <origin xyz="0 0 0.045" rpy="0 0 0"/>
     </joint>
-    <link name="kmriiwa_link_ee">
+    <link name="${robot_name}_link_ee">
     </link>
     <!--Extensions -->
